File: projects/openLRS-APm/openLRS-APM.brd (EAGLE design)
At the start: 43.1 x 20.7 mm, 26 parts, among them IC2 RFM23BPSMD, J1 AVR_SPI_PRG_6PTH, U1 ATMEGA328P, Y1 16MHz

Commit message: Change PPM pin to Timer output.
needed for generating a PPM signal
Connections:
- net PPM: now also U1.13; no longer U1.12
- net SDN: now also U1.11; no longer U1.13
Routing:
- net SDN: track 23.7 -> 22.1 mm
Changed lines of the file:
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@@
 <signal name="SDN">
 <contactref element="IC2" pad="15"/>
-<contactref element="U1" pad="13"/>
 <via x="14.097" y="14.732" extent="1-16" drill="0.6"/>
-<wire x1="13.9954" y1="10.141" x2="15.113" y2="10.141" width="0.4064" layer="1"/>
-<wire x1="15.113" y1="10.141" x2="15.113" y2="13.716" width="0.4064" layer="1"/>
+<wire x1="15.113" y1="11.741" x2="15.113" y2="13.716" width="0.4064" layer="1"/>
 <wire x1="15.113" y1="13.716" x2="14.097" y2="14.732" width="0.4064" layer="1"/>
 <wire x1="14.097" y1="14.732" x2="14.097" y2="12.446" width="0.4064" layer="16"/>
@@
 <wire x1="2.921" y1="13.843" x2="2.921" y2="14.906" width="0.4064" layer="16"/>
 <wire x1="2.921" y1="14.906" x2="1.415" y2="14.906" width="0.4064" layer="16"/>
+<contactref element="U1" pad="11"/>
+<wire x1="13.9954" y1="11.741" x2="15.113" y2="11.741" width="0.4064" layer="1"/>
 </signal>
 <signal name="PPM">
 <contactref element="PPM" pad="1"/>
-<contactref element="U1" pad="12"/>
 <wire x1="5.207" y1="3.81" x2="6.223" y2="4.826" width="0.4064" layer="1"/>
 <via x="6.223" y="4.826" extent="1-16" drill="0.6"/>
@@
 <wire x1="6.223" y1="8.255" x2="10.414" y2="8.255" width="0.4064" layer="16"/>
 <via x="10.414" y="8.255" extent="1-16" drill="0.6"/>
-<wire x1="10.414" y1="8.255" x2="10.414" y2="9.525" width="0.4064" layer="1"/>
-<wire x1="10.414" y1="9.525" x2="13.081" y2="10.922" width="0.4064" layer="1"/>
-<wire x1="13.081" y1="10.922" x2="13.9764" y2="10.922" width="0.4064" layer="1"/>
-<wire x1="13.9764" y1="10.922" x2="13.9954" y2="10.941" width="0.4064" layer="1"/>
 <wire x1="5.207" y1="3.81" x2="5.207" y2="1.905" width="0.4064" layer="1"/>
+<contactref element="U1" pad="13"/>
+<wire x1="10.414" y1="8.255" x2="11.557" y2="9.398" width="0.4064" layer="1"/>
+<wire x1="11.557" y1="9.398" x2="11.557" y2="10.287" width="0.4064" layer="1"/>
+<wire x1="13.9954" y1="10.141" x2="13.227" y2="10.141" width="0.4064" layer="1"/>
+<wire x1="13.227" y1="10.141" x2="12.827" y2="10.541" width="0.4064" layer="1"/>
+<wire x1="12.827" y1="10.541" x2="11.811" y2="10.541" width="0.4064" layer="1"/>
+<wire x1="11.811" y1="10.541" x2="11.557" y2="10.287" width="0.4064" layer="1"/>
 </signal>
 </signals>

Commit message: PPM feedback is cool too!
a few things that we need for rev2. the ppm output should be sampled by
the ICP input.
Connections:
- net PPM: now also U1.12
Routing:
- net PPM: track 16.2 -> 17.3 mm
Changed lines of the file:
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@@
 <wire x1="5.207" y1="3.81" x2="5.207" y2="1.905" width="0.4064" layer="1"/>
 <contactref element="U1" pad="13"/>
-<wire x1="10.414" y1="8.255" x2="11.557" y2="9.398" width="0.4064" layer="1"/>
-<wire x1="11.557" y1="9.398" x2="11.557" y2="10.287" width="0.4064" layer="1"/>
-<wire x1="13.9954" y1="10.141" x2="13.227" y2="10.141" width="0.4064" layer="1"/>
-<wire x1="13.227" y1="10.141" x2="12.827" y2="10.541" width="0.4064" layer="1"/>
-<wire x1="12.827" y1="10.541" x2="11.811" y2="10.541" width="0.4064" layer="1"/>
-<wire x1="11.811" y1="10.541" x2="11.557" y2="10.287" width="0.4064" layer="1"/>
+<wire x1="10.414" y1="8.255" x2="11.43" y2="9.271" width="0.4064" layer="1"/>
+<contactref element="U1" pad="12"/>
+<wire x1="11.43" y1="9.271" x2="11.43" y2="10.795" width="0.4064" layer="1"/>
+<wire x1="11.43" y1="10.795" x2="13.8494" y2="10.795" width="0.4064" layer="1"/>
+<wire x1="13.8494" y1="10.795" x2="13.9954" y2="10.941" width="0.4064" layer="1"/>
+<wire x1="13.8494" y1="10.795" x2="13.8494" y2="10.287" width="0.4064" layer="1"/>
+<wire x1="13.8494" y1="10.287" x2="13.9954" y2="10.141" width="0.4064" layer="1"/>
 </signal>
 </signals>

Commit message: added 3.3v regulator
needed for proper voltages to Atmega.
Parts:
- added C1: 1uF, SparkFun-Capacitors:0805
- added C8: 100n, SparkFun-Capacitors:0805
- added IC1: MCP1703CB, linear:SOT23
Connections:
- new net 3V: C1.1, C8.1, IC1.2, R4.2, U1.18, U1.4, U1.6
- new net 5V: C10.1, C9.1, IC1.3, IC2.5, J1.2, TELEMETRY.P$1, VCC.1
- net GND: now also C1.2, C8.2, IC1.1
- net VCC: no longer C10.1, C9.1, IC2.5, J1.2, R4.2, TELEMETRY.P$1, U1.18, U1.4, U1.6, VCC.1
Routing:
- net VCC: track 92.2 -> 62.6 mm
