File: projects/openLRS-APm/openLRS-APM.sch (EAGLE design)
At the start: 23 parts, among them IC2 RFM23BPSMD, J1 AVR_SPI_PRG_6PTH, U1 ATMEGA328P, X2 SMA-142-0711-821/826, Y1 16MHz

Commit message: Cleaned, Checked, fixed Ground planes
Beefed up Power busses. Fixed the Telemetry Pinout.
Closer to a polished Revision one. Will look into DF-13 PPM signals.
Parts:
- renumbered ICP to PPM, VCC to 5V
Connections:
- net ICP renamed PPM
- removed net SCL: U1.PC5(ADC5/SCL)
- removed net SDA: U1.PC4(ADC4/SDA)
- removed net VCN: U1.PD7(AIN1)
- net DTR: now also TELEMETRY.4; no longer TELEMETRY.6
- net GND: now also TELEMETRY.5, TELEMETRY.6; no longer TELEMETRY.1, TELEMETRY.2
- net RXD: now also TELEMETRY.2; no longer TELEMETRY.4
- net TXD: now also TELEMETRY.3; no longer TELEMETRY.5
- net VCC: now also TELEMETRY.1; no longer TELEMETRY.3
Changed lines of the file:
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@@
 <part name="TELEMETRY" library="con-hirose-df13" deviceset="DF13-6P-1.25" device="H"/>
 <part name="X2" library="con-coax" deviceset="SMA-" device="142-0711-821/826" value="SMA-142-0711-821/826"/>
-<part name="ICP" library="wirepad" deviceset="WIREPAD" device="SMD1,27-254" value=""/>
-<part name="VCC" library="wirepad" deviceset="WIREPAD" device="SMD1,27-254" value=""/>
+<part name="PPM" library="wirepad" deviceset="WIREPAD" device="SMD1,27-254" value=""/>
+<part name="5V" library="wirepad" deviceset="WIREPAD" device="SMD1,27-254" value=""/>
 <part name="GND" library="wirepad" deviceset="WIREPAD" device="SMD1,27-254" value=""/>
 </parts>
@@
 <instance part="TELEMETRY" gate="G$1" x="-10.16" y="104.14" rot="MR0"/>
 <instance part="X2" gate="G1" x="175.26" y="93.98" rot="MR0"/>
-<instance part="ICP" gate="G$1" x="-7.62" y="55.88" smashed="yes">
+<instance part="PPM" gate="G$1" x="-7.62" y="55.88" smashed="yes">
 <attribute name="VALUE" x="-8.763" y="52.578" size="1.778" layer="96"/>
 </instance>
-<instance part="VCC" gate="G$1" x="-7.62" y="53.34" smashed="yes">
+<instance part="5V" gate="G$1" x="-7.62" y="53.34" smashed="yes">
 <attribute name="VALUE" x="-8.763" y="50.038" size="1.778" layer="96"/>
 </instance>
@@
 <nets>
 <net name="GND" class="0">
-<segment>
-<wire x1="-5.08" y1="106.68" x2="-2.54" y2="106.68" width="0.1524" layer="91"/>
-<wire x1="-2.54" y1="106.68" x2="-2.54" y2="109.22" width="0.1524" layer="91"/>
-<wire x1="-2.54" y1="109.22" x2="-5.08" y2="109.22" width="0.1524" layer="91"/>
-<label x="2.54" y="109.22" size="1.778" layer="95"/>
-<junction x="-2.54" y="109.22"/>
-<wire x1="-2.54" y1="109.22" x2="2.54" y2="109.22" width="0.1524" layer="91"/>
-<pinref part="TELEMETRY" gate="G$1" pin="1"/>
-<pinref part="TELEMETRY" gate="G$1" pin="2"/>
-</segment>
 <segment>
 <pinref part="J1" gate="G$1" pin="6"/>
@@
 <label x="-2.54" y="50.8" size="1.778" layer="95"/>
 </segment>
+<segment>
+<pinref part="TELEMETRY" gate="G$1" pin="6"/>
+<wire x1="-5.08" y1="96.52" x2="2.54" y2="96.52" width="0.1524" layer="91"/>
+<label x="2.54" y="96.52" size="1.778" layer="95"/>
+<pinref part="TELEMETRY" gate="G$1" pin="5"/>
+<wire x1="-5.08" y1="99.06" x2="2.54" y2="99.06" width="0.1524" layer="91"/>
+<wire x1="2.54" y1="99.06" x2="2.54" y2="96.52" width="0.1524" layer="91"/>
+</segment>
 </net>
 <net name="VCC" class="0">
-<segment>
-<wire x1="-5.08" y1="104.14" x2="2.54" y2="104.14" width="0.1524" layer="91"/>
-<label x="2.54" y="104.14" size="1.778" layer="95"/>
-<pinref part="TELEMETRY" gate="G$1" pin="3"/>
-</segment>
 <segment>
 <pinref part="SUPPLY1" gate="1" pin="VCC"/>
@@
 </segment>
 <segment>
-<pinref part="VCC" gate="G$1" pin="P"/>
+<pinref part="5V" gate="G$1" pin="P"/>
 <wire x1="-5.08" y1="53.34" x2="-2.54" y2="53.34" width="0.1524" layer="91"/>
 <label x="-2.54" y="53.34" size="1.778" layer="95"/>
 </segment>
+<segment>
+<pinref part="TELEMETRY" gate="G$1" pin="1"/>
+<wire x1="-5.08" y1="109.22" x2="2.54" y2="109.22" width="0.1524" layer="91"/>
+<label x="2.54" y="109.22" size="1.778" layer="95"/>
+</segment>
 </net>
 <net name="RXD" class="0">
-<segment>
-<wire x1="-5.08" y1="101.6" x2="2.54" y2="101.6" width="0.1524" layer="91"/>
-<label x="2.54" y="101.6" size="1.778" layer="95"/>
-<pinref part="TELEMETRY" gate="G$1" pin="4"/>
-</segment>
 <segment>
 <pinref part="U1" gate="G$1" pin="PD0(RXD)"/>
@@
 <label x="93.98" y="68.58" size="1.778" layer="95"/>
 </segment>
+<segment>
+<pinref part="TELEMETRY" gate="G$1" pin="2"/>
+<wire x1="-5.08" y1="106.68" x2="2.54" y2="106.68" width="0.1524" layer="91"/>
+<label x="2.54" y="106.68" size="1.778" layer="95"/>
+</segment>
 </net>
 <net name="TXD" class="0">
-<segment>
-<wire x1="-5.08" y1="99.06" x2="2.54" y2="99.06" width="0.1524" layer="91"/>
-<label x="2.54" y="99.06" size="1.778" layer="95"/>
-<pinref part="TELEMETRY" gate="G$1" pin="5"/>
-</segment>
 <segment>
 <pinref part="U1" gate="G$1" pin="PD1(TXD)"/>
@@
 <label x="93.98" y="66.04" size="1.778" layer="95"/>
 </segment>
+<segment>
+<pinref part="TELEMETRY" gate="G$1" pin="3"/>
+<wire x1="-5.08" y1="104.14" x2="2.54" y2="104.14" width="0.1524" layer="91"/>
+<label x="2.54" y="104.14" size="1.778" layer="95"/>
+</segment>
 </net>
 <net name="DTR" class="0">
-<segment>
-<wire x1="-5.08" y1="96.52" x2="2.54" y2="96.52" width="0.1524" layer="91"/>
-<label x="2.54" y="96.52" size="1.778" layer="95"/>
-<pinref part="TELEMETRY" gate="G$1" pin="6"/>
-</segment>
 <segment>
 <pinref part="C5" gate="G$1" pin="1"/>
 <wire x1="22.86" y1="91.44" x2="20.32" y2="91.44" width="0.1524" layer="91"/>
 <label x="15.24" y="91.44" size="1.778" layer="95"/>
+</segment>
+<segment>
+<pinref part="TELEMETRY" gate="G$1" pin="4"/>
+<wire x1="-5.08" y1="101.6" x2="2.54" y2="101.6" width="0.1524" layer="91"/>
+<label x="2.54" y="101.6" size="1.778" layer="95"/>
 </segment>
 </net>
@@
 </segment>
 </net>
-<net name="SDA" class="0">
-<segment>
-<pinref part="U1" gate="G$1" pin="PC4(ADC4/SDA)"/>
-<wire x1="91.44" y1="81.28" x2="96.52" y2="81.28" width="0.1524" layer="91"/>
-<label x="96.52" y="81.28" size="1.778" layer="95"/>
-</segment>
-</net>
-<net name="SCL" class="0">
-<segment>
-<pinref part="U1" gate="G$1" pin="PC5(ADC5/SCL)"/>
-<wire x1="91.44" y1="78.74" x2="96.52" y2="78.74" width="0.1524" layer="91"/>
-<label x="96.52" y="78.74" size="1.778" layer="95"/>
-</segment>
-</net>
 <net name="MOSI" class="0">
 <segment>
@@
 <pinref part="IC2" gate="G$1" pin="GPIO1"/>
 <wire x1="170.18" y1="68.58" x2="165.1" y2="68.58" width="0.1524" layer="91"/>
-</segment>
-</net>
-<net name="ICP" class="0">
-<segment>
-<pinref part="U1" gate="G$1" pin="PB0(ICP)"/>
-<wire x1="91.44" y1="45.72" x2="93.98" y2="45.72" width="0.1524" layer="91"/>
-<label x="93.98" y="45.72" size="1.778" layer="95"/>
-</segment>
-<segment>
-<pinref part="ICP" gate="G$1" pin="P"/>
-<wire x1="-5.08" y1="55.88" x2="-2.54" y2="55.88" width="0.1524" layer="91"/>
-<label x="-2.54" y="55.88" size="1.778" layer="95"/>
 </segment>
 </net>
@@
 </segment>
 </net>
-<net name="VCN" class="0">
-<segment>
-<pinref part="U1" gate="G$1" pin="PD7(AIN1)"/>
-<wire x1="91.44" y1="50.8" x2="93.98" y2="50.8" width="0.1524" layer="91"/>
-<label x="93.98" y="50.8" size="1.778" layer="95"/>
-</segment>
-</net>
 <net name="SDN" class="0">
 <segment>
@@
 </segment>
 </net>
+<net name="PPM" class="0">
+<segment>
+<pinref part="PPM" gate="G$1" pin="P"/>
+<wire x1="-5.08" y1="55.88" x2="-2.54" y2="55.88" width="0.1524" layer="91"/>
+<label x="-2.54" y="55.88" size="1.778" layer="95"/>
+</segment>
+<segment>
+<pinref part="U1" gate="G$1" pin="PB0(ICP)"/>
+<wire x1="91.44" y1="45.72" x2="93.98" y2="45.72" width="0.1524" layer="91"/>
+<label x="93.98" y="45.72" size="1.778" layer="95"/>
+</segment>
+</net>

Commit message: Changed LED's to 0805.
Prototype Soon. all SMDs are 0805. Hope to find SMA connector
Parts:
- LED1, LED2: device SparkFun-LED:LED1206 -> led:LEDSML0805
- R10, R9: value 220R -> 220
- renumbered 5V to VCC
Changed lines of the file:
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@@
 <grid distance="0.1" unitdist="inch" unit="inch" style="lines" multiple="1" display="no" altdistance="0.01" altunitdist="inch" altunit="inch"/>
 <layers>
-<layer number="1" name="Top" color="4" fill="1" visible="no" active="no"/>
-<layer number="16" name="Bottom" color="1" fill="1" visible="no" active="no"/>
-<layer number="17" name="Pads" color="2" fill="1" visible="no" active="no"/>
-<layer number="18" name="Vias" color="2" fill="1" visible="no" active="no"/>
-<layer number="19" name="Unrouted" color="6" fill="1" visible="no" active="no"/>
-<layer number="20" name="Dimension" color="15" fill="1" visible="no" active="no"/>
-<layer number="21" name="tPlace" color="7" fill="1" visible="no" active="no"/>
-<layer number="22" name="bPlace" color="7" fill="1" visible="no" active="no"/>
-<layer number="23" name="tOrigins" color="15" fill="1" visible="no" active="no"/>
-<layer number="24" name="bOrigins" color="15" fill="1" visible="no" active="no"/>
-<layer number="25" name="tNames" color="7" fill="1" visible="no" active="no"/>
-<layer number="26" name="bNames" color="7" fill="1" visible="no" active="no"/>
-<layer number="27" name="tValues" color="7" fill="1" visible="no" active="no"/>
-<layer number="28" name="bValues" color="7" fill="1" visible="no" active="no"/>
+<layer number="1" name="Top" color="4" fill="1" visible="yes" active="no"/>
+<layer number="16" name="Bottom" color="1" fill="1" visible="yes" active="no"/>
+<layer number="17" name="Pads" color="2" fill="1" visible="yes" active="no"/>
+<layer number="18" name="Vias" color="2" fill="1" visible="yes" active="no"/>
+<layer number="19" name="Unrouted" color="6" fill="1" visible="yes" active="no"/>
+<layer number="20" name="Dimension" color="15" fill="1" visible="yes" active="no"/>
+<layer number="21" name="tPlace" color="7" fill="1" visible="yes" active="no"/>
+<layer number="22" name="bPlace" color="7" fill="1" visible="yes" active="no"/>
+<layer number="23" name="tOrigins" color="15" fill="1" visible="yes" active="no"/>
+<layer number="24" name="bOrigins" color="15" fill="1" visible="yes" active="no"/>
+<layer number="25" name="tNames" color="7" fill="1" visible="yes" active="no"/>
+<layer number="26" name="bNames" color="7" fill="1" visible="yes" active="no"/>
+<layer number="27" name="tValues" color="7" fill="1" visible="yes" active="no"/>
+<layer number="28" name="bValues" color="7" fill="1" visible="yes" active="no"/>
 <layer number="29" name="tStop" color="7" fill="3" visible="no" active="no"/>
 <layer number="30" name="bStop" color="7" fill="6" visible="no" active="no"/>
@@
 <layer number="35" name="tGlue" color="7" fill="4" visible="no" active="no"/>
 <layer number="36" name="bGlue" color="7" fill="5" visible="no" active="no"/>
-<layer number="37" name="tTest" color="7" fill="1" visible="no" active="no"/>
-<layer number="38" name="bTest" color="7" fill="1" visible="no" active="no"/>
+<layer number="37" name="tTest" color="7" fill="1" visible="yes" active="no"/>
+<layer number="38" name="bTest" color="7" fill="1" visible="yes" active="no"/>
 <layer number="39" name="tKeepout" color="4" fill="11" visible="no" active="no"/>
 <layer number="40" name="bKeepout" color="1" fill="11" visible="no" active="no"/>
@@
 <layer number="44" name="Drills" color="7" fill="1" visible="no" active="no"/>
 <layer number="45" name="Holes" color="7" fill="1" visible="no" active="no"/>
-<layer number="46" name="Milling" color="3" fill="1" visible="no" active="no"/>
-<layer number="47" name="Measures" color="7" fill="1" visible="no" active="no"/>
-<layer number="48" name="Document" color="7" fill="1" visible="no" active="no"/>
-<layer number="49" name="Reference" color="7" fill="1" visible="no" active="no"/>
-<layer number="50" name="dxf" color="7" fill="1" visible="no" active="no"/>
-<layer number="51" name="tDocu" color="7" fill="1" visible="no" active="no"/>
-<layer number="52" name="bDocu" color="7" fill="1" visible="no" active="no"/>
-<layer number="53" name="tGND_GNDA" color="7" fill="9" visible="no" active="no"/>
-<layer number="54" name="bGND_GNDA" color="1" fill="9" visible="no" active="no"/>
-<layer number="56" name="wert" color="7" fill="1" visible="no" active="no"/>
-<layer number="57" name="tCAD" color="7" fill="1" visible="no" active="no"/>
+<layer number="46" name="Milling" color="3" fill="1" visible="yes" active="no"/>
+<layer number="47" name="Measures" color="7" fill="1" visible="yes" active="no"/>
+<layer number="48" name="Document" color="7" fill="1" visible="yes" active="no"/>
+<layer number="49" name="Reference" color="7" fill="1" visible="yes" active="no"/>
+<layer number="50" name="dxf" color="7" fill="1" visible="yes" active="no"/>
+<layer number="51" name="tDocu" color="7" fill="1" visible="yes" active="no"/>
+<layer number="52" name="bDocu" color="7" fill="1" visible="yes" active="no"/>
+<layer number="53" name="tGND_GNDA" color="7" fill="9" visible="yes" active="no"/>
+<layer number="54" name="bGND_GNDA" color="1" fill="9" visible="yes" active="no"/>
+<layer number="56" name="wert" color="7" fill="1" visible="yes" active="no"/>
+<layer number="57" name="tCAD" color="7" fill="1" visible="yes" active="no"/>
 <layer number="91" name="Nets" color="2" fill="1" visible="yes" active="yes"/>
 <layer number="92" name="Busses" color="1" fill="1" visible="yes" active="yes"/>
@@
 <part name="J1" library="SparkFun-Connectors" deviceset="AVR_SPI_PRG_6" device="PTH"/>
 <part name="R4" library="SparkFun-Resistors" deviceset="RESISTOR" device="0805-RES" value="10k"/>
-<part name="R9" library="SparkFun-Resistors" deviceset="RESISTOR" device="0805-RES" value="220R"/>
-<part name="R10" library="SparkFun-Resistors" deviceset="RESISTOR" device="0805-RES" value="220R"/>
-<part name="LED1" library="SparkFun-LED" deviceset="LED" device="1206" value="RED"/>
-<part name="LED2" library="SparkFun-LED" deviceset="LED" device="1206" value="GRN"/>
+<part name="R9" library="SparkFun-Resistors" deviceset="RESISTOR" device="0805-RES" value="220"/>
+<part name="R10" library="SparkFun-Resistors" deviceset="RESISTOR" device="0805-RES" value="220"/>
+<part name="LED1" library="led" deviceset="LED" device="SML0805" value="RED"/>
+<part name="LED2" library="led" deviceset="LED" device="SML0805" value="GRN"/>
 <part name="SUPPLY1" library="SparkFun-Aesthetics" deviceset="VCC" device=""/>
 <part name="GND1" library="SparkFun-Aesthetics" deviceset="GND" device=""/>
@@
 <part name="X2" library="con-coax" deviceset="SMA-" device="142-0711-821/826" value="SMA-142-0711-821/826"/>
 <part name="PPM" library="wirepad" deviceset="WIREPAD" device="SMD1,27-254" value=""/>
-<part name="5V" library="wirepad" deviceset="WIREPAD" device="SMD1,27-254" value=""/>
+<part name="VCC" library="wirepad" deviceset="WIREPAD" device="SMD1,27-254" value=""/>
 <part name="GND" library="wirepad" deviceset="WIREPAD" device="SMD1,27-254" value=""/>
 </parts>
@@
 <instance part="TELEMETRY" gate="G$1" x="-10.16" y="104.14" rot="MR0"/>
 <instance part="X2" gate="G1" x="175.26" y="93.98" rot="MR0"/>
-<instance part="PPM" gate="G$1" x="-7.62" y="55.88" smashed="yes">
-<attribute name="VALUE" x="-8.763" y="52.578" size="1.778" layer="96"/>
-</instance>
-<instance part="5V" gate="G$1" x="-7.62" y="53.34" smashed="yes">
-<attribute name="VALUE" x="-8.763" y="50.038" size="1.778" layer="96"/>
-</instance>
-<instance part="GND" gate="G$1" x="-7.62" y="50.8" smashed="yes">
-<attribute name="VALUE" x="-8.763" y="47.498" size="1.778" layer="96"/>
-</instance>
+<instance part="PPM" gate="G$1" x="-7.62" y="55.88" smashed="yes"/>
+<instance part="VCC" gate="G$1" x="-7.62" y="53.34" smashed="yes"/>
+<instance part="GND" gate="G$1" x="-7.62" y="50.8" smashed="yes"/>
 </instances>
 <busses>
@@
 </segment>
 <segment>
-<pinref part="5V" gate="G$1" pin="P"/>
+<pinref part="VCC" gate="G$1" pin="P"/>
 <wire x1="-5.08" y1="53.34" x2="-2.54" y2="53.34" width="0.1524" layer="91"/>
 <label x="-2.54" y="53.34" size="1.778" layer="95"/>
