File: projects/openLRS-APM/openLRS-APM.sch (EAGLE design)
At the start: 26 parts, among them IC1 MCP1703CB, IC2 RFM23BPSMD, J1 AVR_SPI_PRG_6PTH, U1 ATMEGA328P, Y1 16MHz

Commit message: Initial Rev2 Commit
Rearranged for shrink wrapping, fixed voltage levels. may need routing
touch up.
Parts:
- removed C2: 100n, SparkFun-Capacitors:CAP0805
Connections:
- removed net SDN: IC2.SDN, U1.PD7(AIN1)
- removed net VCC: C2.1, C7.1, R8.2
- net 3V: now also C7.1, R8.2
- net GND: now also IC2.SDN; no longer C2.2
- net N$1: now also IC2.GPIO1; no longer IC2.GPIO0
- net N$2: now also IC2.GPIO0; no longer IC2.GPIO1
Changed lines of the file:
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@@
 <part name="GND2" library="SparkFun-Aesthetics" deviceset="GND" device=""/>
 <part name="GND4" library="SparkFun-Aesthetics" deviceset="GND" device=""/>
-<part name="SUPPLY4" library="SparkFun-Aesthetics" deviceset="VCC" device=""/>
 <part name="C3" library="SparkFun-Capacitors" deviceset="CAP" device="0805" value="12pF"/>
 <part name="C4" library="SparkFun-Capacitors" deviceset="CAP" device="0805" value="12pF"/>
@@
 <part name="C10" library="SparkFun-Capacitors" deviceset="CAP" device="0805" value="100n"/>
 <part name="R8" library="SparkFun-Resistors" deviceset="RESISTOR" device="0805-RES" value="1k"/>
-<part name="SUPPLY5" library="SparkFun-Aesthetics" deviceset="VCC" device=""/>
 <part name="C6" library="SparkFun-Capacitors" deviceset="CAP" device="0805" value="100n"/>
 <part name="GND7" library="SparkFun-Aesthetics" deviceset="GND" device=""/>
-<part name="C2" library="SparkFun-Capacitors" deviceset="CAP" device="0805" value="100n"/>
 <part name="TELEMETRY" library="con-hirose-df13" deviceset="DF13-6P-1.25" device="H"/>
 <part name="PPM" library="wirepad" deviceset="WIREPAD" device="SMD1,27-254" value=""/>
@@
 <instance part="GND2" gate="1" x="38.1" y="25.4"/>
 <instance part="GND4" gate="1" x="111.76" y="20.32"/>
-<instance part="SUPPLY4" gate="1" x="30.48" y="50.8"/>
 <instance part="C3" gate="G$1" x="25.4" y="66.04" rot="R270"/>
 <instance part="C4" gate="G$1" x="25.4" y="60.96" rot="R270"/>
@@
 <instance part="C10" gate="G$1" x="129.54" y="96.52"/>
 <instance part="R8" gate="G$1" x="106.68" y="63.5" rot="R90"/>
-<instance part="SUPPLY5" gate="1" x="106.68" y="71.12"/>
 <instance part="C6" gate="G$1" x="30.48" y="76.2" rot="R90"/>
 <instance part="GND7" gate="1" x="25.4" y="71.12"/>
-<instance part="C2" gate="G$1" x="22.86" y="43.18"/>
 <instance part="TELEMETRY" gate="G$1" x="-10.16" y="104.14" rot="MR0"/>
 <instance part="PPM" gate="G$1" x="-7.62" y="55.88" smashed="yes"/>
@@
 <junction x="127" y="93.98"/>
 <junction x="137.16" y="71.12"/>
+<pinref part="IC2" gate="G$1" pin="SDN"/>
+<wire x1="139.7" y1="73.66" x2="137.16" y2="73.66" width="0.1524" layer="91"/>
+<wire x1="137.16" y1="73.66" x2="137.16" y2="71.12" width="0.1524" layer="91"/>
 </segment>
 <segment>
@@
 <wire x1="38.1" y1="40.64" x2="30.48" y2="40.64" width="0.1524" layer="91"/>
 <junction x="38.1" y="40.64"/>
-<pinref part="C2" gate="G$1" pin="2"/>
-<wire x1="30.48" y1="40.64" x2="22.86" y2="40.64" width="0.1524" layer="91"/>
-<junction x="30.48" y="40.64"/>
 </segment>
 <segment>
@@
 </segment>
 </net>
-<net name="VCC" class="0">
-<segment>
-<pinref part="C7" gate="G$1" pin="1"/>
-<wire x1="30.48" y1="48.26" x2="30.48" y2="50.8" width="0.1524" layer="91"/>
-<pinref part="SUPPLY4" gate="1" pin="VCC"/>
-<pinref part="C2" gate="G$1" pin="1"/>
-<wire x1="30.48" y1="48.26" x2="22.86" y2="48.26" width="0.1524" layer="91"/>
-<junction x="30.48" y="48.26"/>
-</segment>
-<segment>
-<pinref part="R8" gate="G$1" pin="2"/>
-<pinref part="SUPPLY5" gate="1" pin="VCC"/>
-<wire x1="106.68" y1="68.58" x2="106.68" y2="71.12" width="0.1524" layer="91"/>
-</segment>
-</net>
 <net name="RXD" class="0">
 <segment>
@@
 <pinref part="IC2" gate="G$1" pin="TXANT"/>
 <wire x1="165.1" y1="76.2" x2="167.64" y2="76.2" width="0.1524" layer="91"/>
-<wire x1="167.64" y1="76.2" x2="167.64" y2="71.12" width="0.1524" layer="91"/>
-<pinref part="IC2" gate="G$1" pin="GPIO0"/>
-<wire x1="167.64" y1="71.12" x2="165.1" y2="71.12" width="0.1524" layer="91"/>
+<wire x1="167.64" y1="76.2" x2="167.64" y2="68.58" width="0.1524" layer="91"/>
+<pinref part="IC2" gate="G$1" pin="GPIO1"/>
+<wire x1="167.64" y1="68.58" x2="165.1" y2="68.58" width="0.1524" layer="91"/>
 </segment>
 </net>
@@
 <pinref part="IC2" gate="G$1" pin="RXANT"/>
 <wire x1="165.1" y1="78.74" x2="170.18" y2="78.74" width="0.1524" layer="91"/>
-<wire x1="170.18" y1="78.74" x2="170.18" y2="68.58" width="0.1524" layer="91"/>
-<pinref part="IC2" gate="G$1" pin="GPIO1"/>
-<wire x1="170.18" y1="68.58" x2="165.1" y2="68.58" width="0.1524" layer="91"/>
+<wire x1="170.18" y1="78.74" x2="170.18" y2="71.12" width="0.1524" layer="91"/>
+<pinref part="IC2" gate="G$1" pin="GPIO0"/>
+<wire x1="170.18" y1="71.12" x2="165.1" y2="71.12" width="0.1524" layer="91"/>
 </segment>
 </net>
@@
 <pinref part="LED1" gate="G$1" pin="A"/>
 <wire x1="106.68" y1="35.56" x2="106.68" y2="33.02" width="0.1524" layer="91"/>
-</segment>
-</net>
-<net name="SDN" class="0">
-<segment>
-<pinref part="IC2" gate="G$1" pin="SDN"/>
-<wire x1="139.7" y1="73.66" x2="137.16" y2="73.66" width="0.1524" layer="91"/>
-<label x="132.08" y="73.66" size="1.778" layer="95"/>
-</segment>
-<segment>
-<pinref part="U1" gate="G$1" pin="PD7(AIN1)"/>
-<wire x1="91.44" y1="50.8" x2="93.98" y2="50.8" width="0.1524" layer="91"/>
-<label x="93.98" y="50.8" size="1.778" layer="95"/>
 </segment>
 </net>
@@
 <pinref part="C8" gate="G$1" pin="1"/>
 </segment>
-</net>
+<segment>
+<pinref part="C7" gate="G$1" pin="1"/>
+<wire x1="30.48" y1="48.26" x2="30.48" y2="50.8" width="0.1524" layer="91"/>
+<label x="30.48" y="50.8" size="1.778" layer="95"/>
+</segment>
+<segment>
+<pinref part="R8" gate="G$1" pin="2"/>
+<wire x1="106.68" y1="68.58" x2="106.68" y2="71.12" width="0.1524" layer="91"/>
+<label x="106.68" y="71.12" size="1.778" layer="95"/>
+</segment>
+</net>

Commit message: Initial 32u4 USB dongle version
Parts:
- removed C7: 100n, SparkFun-Capacitors:CAP0805
- removed GND, PPM, VCC: WIREPADSMD1,27-254, wirepad:WIREPADSMD1,27-254
- removed R8: 1k, SparkFun-Resistors:RESISTOR0805-RES
- removed TELEMETRY: DF13-6P-1.25H, con-hirose-df13:DF13-6P-1.25H
- removed U1: ATMEGA328P, SparkFun-DigitalIC:ATMEGA328_SMT
- added C11: 100n, SparkFun-Capacitors:CAP0805
- added C2: 1uF, SparkFun-Capacitors:CAP0805
- added JP1: USB-A-H, SparkFun-Connectors:USB-A-H
- added MCU1: ATMEGA32U4TQFP, SparkFun-DigitalIC:ATMEGA32U4TQFP
- added R1, R2: 22, SparkFun-Resistors:RESISTOR0805-RES
- C5: value 100n -> 1uF
- J1: value AVR_SPI_PRG_6PTH -> CON_HEADER_PRG_AVR_ICSP-SMD; device SparkFun-Connectors:AVR_SPI_PRG_6PTH -> dp_devices:CON_HEADER_PRG_AVR_ICSP-SMD
Connections:
- removed net DTR: C5.1, TELEMETRY.4
- removed net N$14: C6.2, U1.AREF
- removed net PPM: PPM.P, U1.PB0(ICP), U1.PB1(OC1A)
- removed net RF_CS: IC2.NSEL, R8.1, U1.PD4(XCK/T0)
- removed net RF_IRQ: IC2.NIRQ, U1.PD2(INT0)
- removed net RXD: TELEMETRY.2, U1.PD0(RXD)
- removed net TXD: TELEMETRY.3, U1.PD1(TXD)
- new net CS: IC2.NSEL, MCU1.PB6(ADC13)
- new net D_N: MCU1.D-, R2.1
- new net D_P: MCU1.D+, R1.1
- new net IRQ: IC2.NIRQ, MCU1.PD0(SCL)
- new net N$3: C6.2, MCU1.AREF
- new net R_N: JP1.D+, R2.2
- new net R_P: JP1.D-, R1.2
- new net UCAP: C5.1, MCU1.UCAP
- net /RESET: now also J1.RST, MCU1.!RESET; no longer C5.2, J1.5, U1.PC6(/RESET)
- net 3V: now also MCU1.AVCC@24, MCU1.AVCC@44, MCU1.VCC@14, MCU1.VCC@34; no longer C7.1, R8.2, U1.AVCC, U1.VCC@1, U1.VCC@2
- net 5V: now also C11.1, C2.1, J1.+V, JP1.GND, MCU1.UVCC, MCU1.VBUS; no longer J1.2, TELEMETRY.1, VCC.P
- net GND: now also C11.2, C2.2, C5.2, J1.GND, JP1.VBUS, MCU1.GND@15, MCU1.GND@23, MCU1.GND@35, MCU1.GND@43, MCU1.UGND; no longer C7.2, GND.P, J1.6, TELEMETRY.5, TELEMETRY.6, U1.AGND, U1.GND@1, U1.GND@2
- net MISO: now also J1.MISO, MCU1.PB3(MISO); no longer J1.1, U1.PB4(MISO)
- net MOSI: now also J1.MOSI, MCU1.PB2(MOSI); no longer J1.4, U1.PB3(MOSI/OC2)
- net N$1: now also IC2.TXON; no longer IC2.TXANT
- net N$11: now also MCU1.XTAL1; no longer U1.PB6(XTAL1/TOSC1)
- net N$12: now also MCU1.XTAL2; no longer U1.PB7(XTAL2/TOSC2)
- net N$2: now also IC2.RXON; no longer IC2.RXANT
- net N$7: now also MCU1.PB4(ADC11); no longer U1.PD6(AIN0)
- net N$8: now also MCU1.PD7(ADC10); no longer U1.PD5(T1)
- net SCK: now also J1.SCK, MCU1.PB1(SCK); no longer J1.3, U1.PB5(SCK)
Other:
- moved on the sheet: C10, C3, C4, C5, C6, C9, IC2, SMA, Y1
